File: GAR_Vehicle_Controller_RevA/03_RC_RECEIVER.kicad_sch (KiCad schematic)
At the start: 0 parts

Commit message: Draw first draft of the RC receiver sheet
03_RC_RECEIVER now has the J1 header, 0R series links, an unfitted
2N7002 inverter with a 0R bypass, supply bypass caps, and four test
points, ending in the RC_UART_RX / RC_UART_TX hierarchical labels.
The top sheet gains matching sheet pins and its sheet symbols are moved
onto the 2.54 mm grid. ERC reports four expected items until the other
sheets exist.
Parts:
- added C1: 100n, Capacitor_SMD:C_0805_2012Metric, symbol Device:C
- added C2: 10u, Capacitor_SMD:C_0805_2012Metric, symbol Device:C
- added J1: ER4 receiver, Connector_PinHeader_2.54mm:PinHeader_1x04_P2.54mm_Vertical, symbol Connector_Generic:Conn_01x04
- added Q1: 2N7002, Package_TO_SOT_SMD:SOT-23, symbol Transistor_FET:Q_NMOS_GSD
- added R1, R2, R3: 0R, Resistor_SMD:R_0805_2012Metric, symbol Device:R
- added R4: 10k, Resistor_SMD:R_0805_2012Metric, symbol Device:R
- added TP1, TP2, TP3, TP4: TestPoint, TestPoint:TestPoint_Pad_D1.5mm, symbol Connector:TestPoint
Connections:
- new net: J1.4 (Pin_4), R2.1
- new net: J1.1 (Pin_1), R1.1
- new net: Q1.1 (G), R1.2, R3.1
- new net +3V3: R4.1
- new net +5V_LOGIC: C1.1, C2.1, J1.2 (Pin_2), TP3.1
- new net GND: C1.2, C2.2, J1.3 (Pin_3), Q1.2 (S), TP4.1
- new net RC_UART_RX: Q1.3 (D), R3.2, R4.2, TP1.1
- new net RC_UART_TX: R2.2, TP2.1
Other:
- note added: "If fitted, remove R3."
- note added: "J1 pin order is a proposal: 1 = serial line A, 2 = +5 V, 3 = GND, 4 = serial line B."
- note added: "Q1 + R4: optional inverter / 3.3 V level shifter, not fitted."
- note added: "R1, R2: 0R links. Remove to isolate a line during bring-up."
- note added: "RC receiver interface: RadioMaster ER4 (ExpressLRS), SBUS or CRSF."
- note added: "Receiver supply bypass, place next to J1."
- note added: "TODO: confirm on a real ER4 which channel pins carry serial and which line is TX / RX."
- note added: "The receiver is off-board and connects to J1 with four jumper wires. See docs/interface_notes.md."
